Commit message: add gazebo

File: src/urdf_gazebo_demo/xacro/car.xacro (robot description, xacro)
@@ -1,3 +1,4 @@
 <robot xmlns:xacro="http://www.ros.org/wiki/xacro" name="mycar">
+    <xacro:include filename="head.xacro"/>
     <xacro:include filename="car_base.xacro"/>
     <xacro:include filename="car_camera.xacro"/>

File: src/urdf_gazebo_demo/xacro/car_base.xacro (robot description, xacro)
@@ -4,4 +4,7 @@
     <xacro:property name="base_radius" value="0.1"/>
     <xacro:property name="base_length" value="0.08"/>
+    <xacro:property name="base_mass" value="2"/>
+    <xacro:property name="wheel_mass" value="0.05"/>
+    <xacro:property name="small_wheel_mass" value="0.01"/>
     <xacro:property name="lidi" value="0.015"/>
     <xacro:property name="base_joint_z" value="${base_length / 2 + lidi}"/>
@@ -23,5 +26,17 @@
             </material>
         </visual>
+        <collision>
+            <geometry>
+                <cylinder radius="${base_radius}" length="${base_length}" />
+            </geometry>
+            <origin xyz="0 0 0" rpy="0 0 0" />
+        </collision>
+        <xacro:cylinder_inertial_matrix m="${base_mass}" r="${base_radius}" h="${base_length}" />
     </link>
+    <gazebo reference="base_link">
+        <material>
+        Gazebo/Yellow
+        </material>
+    </gazebo>
     <joint name="base_link2base_footprint" type="fixed">
         <parent link="base_footprint"/>
@@ -49,5 +64,17 @@
                 </material>
             </visual>
+            <collision>
+                <geometry>
+                    <cylinder radius="${wheel_radius}" length="${wheel_length}" />
+                </geometry>
+                <origin xyz="0 0 0" rpy="${PI /2} 0 0" />
+            </collision>
+            <xacro:cylinder_inertial_matrix m="${wheel_mass}" r="${wheel_radius}" h="${wheel_length}" />
         </link>
+        <gazebo reference="${wheel_name}_wheel">
+            <material>
+                Gazebo/Red
+            </material>
+        </gazebo>
         <joint name="${wheel_name}2link" type="continuous">
             <parent link="base_link" />
@@ -70,5 +97,17 @@
                 </material>
             </visual>
+            <collision>
+                <geometry>
+                    <sphere radius="${small_wheel_radius}" />
+                </geometry>
+                <origin xyz="0 0 0" rpy="0 0 0" />
+            </collision>
+            <xacro:sphere_inertial_matrix m="${small_wheel_mass}" r="${small_wheel_radius}" />
         </link>
+        <gazebo reference="${small_wheel_name}_wheel">
+            <material>
+                Gazebo/Red
+            </material>
+        </gazebo>
         <joint name="${small_wheel_name}2link" type="continuous">
             <parent link="base_link" />

File: src/urdf_gazebo_demo/xacro/car_laser.xacro (robot description, xacro)
@@ -4,6 +4,8 @@
     <xacro:property name="support_radius" value="0.01"/>
     <xacro:property name="support_length" value="0.1"/>
+    <xacro:property name="support_mass" value="0.1"/>
     <xacro:property name="laser_radius" value="0.03"/>
     <xacro:property name="laser_length" value="0.05"/>
+    <xacro:property name="laser_mass" value="0.05"/>
     <xacro:property name="joint_support_x" value="0"/>
     <xacro:property name="joint_support_y" value="0"/>
@@ -22,5 +24,17 @@
             </material>
         </visual>
+        <collision>
+            <geometry>
+                <cylinder radius="${support_radius}" length="${support_length}"/>
+            </geometry>
+            <origin xyz="0.0 0.0 0.0" rpy="0.0 0.0 0.0"/>
+        </collision>
+        <xacro:cylinder_inertial_matrix m="${support_mass}" r="${support_radius}" h="${support_length}" />
     </link>
+    <gazebo reference="support">
+        <material>
+            Gazebo/Gray
+        </material>
+    </gazebo>
     <joint name="support2base" type="fixed">
         <parent link="base_link"/>
@@ -36,5 +50,17 @@
             <material name="black"/>
         </visual>
+        <collision>
+            <geometry>
+                <cylinder radius="${laser_radius}" length="${laser_length}" />
+            </geometry>
+            <origin xyz="0.0 0.0 0.0" rpy="0.0 0.0 0.0" />
+        </collision>
+        <xacro:cylinder_inertial_matrix m="${laser_mass}" r="${laser_radius}" h="${laser_length}" />
     </link>
+    <gazebo reference="laser">
+        <material>
+            Gazebo/Black
+        </material>
+    </gazebo>
     <joint name="laser2support" type="fixed">
         <parent link="support" />

Commit message: add simulator

File: src/urdf_gazebo_demo/xacro/car.xacro (robot description, xacro)
@@ -4,3 +4,7 @@
     <xacro:include filename="car_camera.xacro"/>
     <xacro:include filename="car_laser.xacro"/>
+    <xacro:include filename="gazebo/move.xacro"/>
+    <xacro:include filename="gazebo/laser.xacro"/>
+    <xacro:include filename="gazebo/camera.xacro"/>
+    <xacro:include filename="gazebo/kinect.xacro"/>
 </robot>

File: src/urdf_gazebo_demo/xacro/car_base.xacro (robot description, xacro)
@@ -43,9 +43,4 @@
         <child link="base_link"/>
         <origin xyz="0 0 ${lidi+ base_length / 2}" />
-    </joint>
-    <joint name="link2footprint" type="fixed">
-        <parent link="base_footprint"/>
-        <child link="base_link"/>
-        <origin xyz="0 0 0.05 " rpy="0 0 0" />
     </joint>
     <xacro:property name="wheel_radius" value="0.02" />
