Commit message: modify gazebo

File: src/urdf_gazebo_demo/xacro/car_base.xacro (robot description, xacro)
@@ -9,4 +9,10 @@
     <xacro:property name="lidi" value="0.015"/>
     <xacro:property name="base_joint_z" value="${base_length / 2 + lidi}"/>
+    <xacro:property name="wheel_radius" value="0.02" />
+    <xacro:property name="wheel_length" value="0.02" />
+    <xacro:property name="PI" value="3.1415927" />
+    <xacro:property name="wheel_joint_z" value="${-1* (base_length / 2 + lidi - wheel_radius)}" />
+    <xacro:property name="small_wheel_radius" value="0.015"/>
+    <xacro:property name="small_joint_z" value="${-(0.5*base_length+lidi-small_wheel_radius)}"/>
     <link name="base_footprint">
         <visual>
@@ -42,10 +48,7 @@
         <parent link="base_footprint"/>
         <child link="base_link"/>
-        <origin xyz="0 0 ${lidi+ base_length / 2}" />
+        <!-- <origin xyz="0 0 0" /> -->
+        <origin xyz="0 0 ${base_joint_z}" />
     </joint>
-    <xacro:property name="wheel_radius" value="0.02" />
-    <xacro:property name="wheel_length" value="0.02" />
-    <xacro:property name="PI" value="3.1415927" />
-    <xacro:property name="wheel_joint_z" value="${-1* (base_length / 2 + lidi - wheel_radius)}" />
     <xacro:macro name="wheel_func" params="wheel_name flag">
         <link name="${wheel_name}_wheel">
@@ -75,10 +78,8 @@
             <parent link="base_link" />
             <child link="${wheel_name}_wheel" />
-            <origin xyz="0 ${0.1*flag} ${wheel_joint_z}" rpy="0 0 0" />
-            <axis xyz="0 0 0.5" />
+            <origin xyz="0 ${base_radius*flag} ${-(lidi+base_length/2-wheel_radius)}" rpy="0 0 0" />
+            <axis xyz="0 1 0" />
         </joint>
     </xacro:macro>
-    <xacro:property name="small_wheel_radius" value="0.015"/>
-    <xacro:property name="small_joint_z" value="${(0.5*base_length+lidi-small_wheel_radius)*-1}"/>
     <xacro:macro name="small_wheel_func" params="small_wheel_name flag">
         <link name="${small_wheel_name}_wheel">
@@ -108,6 +109,7 @@
             <parent link="base_link" />
             <child link="${small_wheel_name}_wheel" />
-            <origin xyz="${0.08*flag} 0 ${small_joint_z}" rpy="0 0 0" />
-            <axis xyz="0 0 0.5" />
+            <origin xyz="${(base_radius-small_wheel_radius)*flag} 0 ${-(base_length+lidi-small_wheel_radius)/2}" rpy="0 0 0" />
+            <!-- <origin xyz="${(base_radius-small_wheel_radius)*flag} 0 ${small_joint_z}" rpy="0 0 0" /> -->
+            <axis xyz="1 1 1" />
         </joint>
     </xacro:macro>
